File: ai03-pcb-guide.kicad_pcb (KiCad board)
At the start: 2 copper layers, 76.2 x 38.1 mm, 24 parts, among them SW1 SW_Push, U1 ATmega32U4-AU, Y1 16MHz

Commit message: Route components
Parts:
- SW1, USB1: moved to B.Cu
- moved F1 14.7 mm to (44.5, 92.3)
- moved R1 2.38 mm to (47.6, 89.6)
- moved R2 2.38 mm to (50.0, 89.6)
- turned C4 to 90 degrees
- turned D1 to 90 degrees
- turned D2 to 90 degrees
- turned D3 to 90 degrees
- turned D4 to 90 degrees
- turned SW1 to 180 degrees
Connections:
- Y1 pad 2: Net-(Y1-Pad2) -> GND
- Y1 pad 4: Net-(Y1-Pad2) -> GND
Routing:
- net GND: track 0.00 -> 129.1 mm, vias 0 -> 5
- net +5V: track 0.00 -> 76.4 mm, vias 0 -> 4
- net Net-(R3-Pad2): track 0.00 -> 29.8 mm, vias 0 -> 2
- net Net-(R1-Pad1): track 0.00 -> 23.9 mm
- net Net-(R2-Pad1): track 0.00 -> 21.9 mm
- net ROW1: track 0.00 -> 19.8 mm
- net ROW0: track 0.00 -> 19.8 mm
- net COL1: track 0.00 -> 19.1 mm
- net COL0: track 0.00 -> 19.0 mm
- net Net-(C5-Pad1): track 0.00 -> 12.4 mm
- net Net-(C4-Pad1): track 0.00 -> 9.43 mm
- net Net-(D4-Pad2): track 0.00 -> 6.79 mm
- net Net-(D3-Pad2): track 0.00 -> 6.62 mm
- net Net-(D2-Pad2): track 0.00 -> 6.62 mm
- net Net-(D1-Pad2): track 0.00 -> 6.62 mm
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Other:
- net class Default: trace_width 0.25 -> 0.254
- net class Power added: clearance 0.2, trace_width 0.381, via_dia 0.8, via_drill 0.4

Commit message: Route to switches
Connections:
- U1 pad 27: Net-(U1-Pad27) -> COL0
- U1 pad 28: Net-(U1-Pad28) -> COL1
- U1 pad 29: Net-(U1-Pad29) -> ROW0
- U1 pad 30: Net-(U1-Pad30) -> ROW1
- Y1 pad 2: GND -> Net-(Y1-Pad2)
- Y1 pad 4: GND -> Net-(Y1-Pad2)
Routing:
- net ROW1: track 19.8 -> 65.7 mm
- net ROW0: track 19.8 -> 46.6 mm
- net COL0: track 19.0 -> 42.1 mm
- net COL1: track 19.1 -> 32.2 mm
Changed lines of the file:
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@@
     (thickness 1.6)
     (drawings 8)
-    (tracks 161)
+    (tracks 174)
     (zones 0)
     (modules 24)
-    (nets 49)
+    (nets 46)
   )
   (page A4)
@@
   (net 28 "Net-(U1-Pad32)")
   (net 29 "Net-(U1-Pad31)")
-  (net 30 "Net-(U1-Pad30)")
-  (net 31 "Net-(U1-Pad29)")
-  (net 32 "Net-(U1-Pad28)")
-  (net 33 "Net-(U1-Pad27)")
-  (net 34 "Net-(U1-Pad26)")
-  (net 35 "Net-(U1-Pad25)")
-  (net 36 "Net-(U1-Pad22)")
-  (net 37 "Net-(U1-Pad21)")
-  (net 38 "Net-(U1-Pad20)")
-  (net 39 "Net-(U1-Pad19)")
-  (net 40 "Net-(U1-Pad18)")
-  (net 41 "Net-(U1-Pad12)")
-  (net 42 "Net-(U1-Pad11)")
-  (net 43 "Net-(U1-Pad10)")
-  (net 44 "Net-(U1-Pad9)")
-  (net 45 "Net-(U1-Pad8)")
-  (net 46 "Net-(U1-Pad1)")
-  (net 47 "Net-(USB1-Pad6)")
-  (net 48 "Net-(USB1-Pad2)")
+  (net 30 "Net-(U1-Pad26)")
+  (net 31 "Net-(U1-Pad25)")
+  (net 32 "Net-(U1-Pad22)")
+  (net 33 "Net-(U1-Pad21)")
+  (net 34 "Net-(U1-Pad20)")
+  (net 35 "Net-(U1-Pad19)")
+  (net 36 "Net-(U1-Pad18)")
+  (net 37 "Net-(U1-Pad12)")
+  (net 38 "Net-(U1-Pad11)")
+  (net 39 "Net-(U1-Pad10)")
+  (net 40 "Net-(U1-Pad9)")
+  (net 41 "Net-(U1-Pad8)")
+  (net 42 "Net-(U1-Pad1)")
+  (net 43 "Net-(USB1-Pad6)")
+  (net 44 "Net-(USB1-Pad2)")
+  (net 45 "Net-(Y1-Pad2)")
   (net_class Default "This is the default net class."
     (clearance 0.2)
@@
     (add_net "Net-(U1-Pad25)")
     (add_net "Net-(U1-Pad26)")
-    (add_net "Net-(U1-Pad27)")
-    (add_net "Net-(U1-Pad28)")
-    (add_net "Net-(U1-Pad29)")
-    (add_net "Net-(U1-Pad30)")
     (add_net "Net-(U1-Pad31)")
     (add_net "Net-(U1-Pad32)")
@@
     (add_net "Net-(USB1-Pad2)")
     (add_net "Net-(USB1-Pad6)")
+    (add_net "Net-(Y1-Pad2)")
     (add_net ROW0)
     (add_net ROW1)
@@
     (fp_line (start 2.1 1.7) (end -2.1 1.7) (layer B.CrtYd) (width 0.05))
     (pad 4 smd rect (at -1.1 0.85 180) (size 1.4 1.2) (layers B.Cu B.Paste B.Mask)
-      (net 1 GND))
+      (net 45 "Net-(Y1-Pad2)"))
     (pad 3 smd rect (at 1.1 0.85 180) (size 1.4 1.2) (layers B.Cu B.Paste B.Mask)
       (net 4 "Net-(C5-Pad1)"))
     (pad 2 smd rect (at 1.1 -0.85 180) (size 1.4 1.2) (layers B.Cu B.Paste B.Mask)
-      (net 1 GND))
+      (net 45 "Net-(Y1-Pad2)"))
     (pad 1 smd rect (at -1.1 -0.85 180) (size 1.4 1.2) (layers B.Cu B.Paste B.Mask)
       (net 3 "Net-(C4-Pad1)"))
@@
     (fp_line (start 3.25 1.25) (end 5.5 1.25) (layer B.CrtYd) (width 0.15))
     (pad 6 thru_hole oval (at 0 3.65 270) (size 2.7 1.7) (drill oval 1.9 0.7) (layers *.Cu *.Mask)
-      (net 47 "Net-(USB1-Pad6)"))
+      (net 43 "Net-(USB1-Pad6)"))
     (pad 6 thru_hole oval (at 0 -3.65 270) (size 2.7 1.7) (drill oval 1.9 0.7) (layers *.Cu *.Mask)
-      (net 47 "Net-(USB1-Pad6)"))
+      (net 43 "Net-(USB1-Pad6)"))
     (pad 6 thru_hole oval (at 4.5 -3.65 270) (size 2.7 1.7) (drill oval 1.9 0.7) (layers *.Cu *.Mask)
-      (net 47 "Net-(USB1-Pad6)"))
+      (net 43 "Net-(USB1-Pad6)"))
     (pad 6 thru_hole oval (at 4.5 3.65 270) (size 2.7 1.7) (drill oval 1.9 0.7) (layers *.Cu *.Mask)
-      (net 47 "Net-(USB1-Pad6)"))
+      (net 43 "Net-(USB1-Pad6)"))
     (pad 5 smd rect (at 4.5 1.6 270) (size 2.25 0.5) (layers B.Cu B.Paste B.Mask)
       (net 12 VCC))
@@
       (net 17 D+))
     (pad 2 smd rect (at 4.5 -0.8 270) (size 2.25 0.5) (layers B.Cu B.Paste B.Mask)
-      (net 48 "Net-(USB1-Pad2)"))
+      (net 44 "Net-(USB1-Pad2)"))
     (pad 1 smd rect (at 4.5 -1.6 270) (size 2.25 0.5) (layers B.Cu B.Paste B.Mask)
       (net 1 GND))
@@
       (net 29 "Net-(U1-Pad31)"))
     (pad 30 smd rect (at 5.7 1.6) (size 1.5 0.55) (layers B.Cu B.Paste B.Mask)
-      (net 30 "Net-(U1-Pad30)"))
+      (net 9 ROW1))
     (pad 29 smd rect (at 5.7 0.8) (size 1.5 0.55) (layers B.Cu B.Paste B.Mask)
-      (net 31 "Net-(U1-Pad29)"))
+      (net 7 ROW0))
     (pad 28 smd rect (at 5.7 0) (size 1.5 0.55) (layers B.Cu B.Paste B.Mask)
-      (net 32 "Net-(U1-Pad28)"))
+      (net 14 COL1))
     (pad 27 smd rect (at 5.7 -0.8) (size 1.5 0.55) (layers B.Cu B.Paste B.Mask)
-      (net 33 "Net-(U1-Pad27)"))
+      (net 13 COL0))
     (pad 26 smd rect (at 5.7 -1.6) (size 1.5 0.55) (layers B.Cu B.Paste B.Mask)
-      (net 34 "Net-(U1-Pad26)"))
+      (net 30 "Net-(U1-Pad26)"))
     (pad 25 smd rect (at 5.7 -2.4) (size 1.5 0.55) (layers B.Cu B.Paste B.Mask)
-      (net 35 "Net-(U1-Pad25)"))
+      (net 31 "Net-(U1-Pad25)"))
     (pad 24 smd rect (at 5.7 -3.2) (size 1.5 0.55) (layers B.Cu B.Paste B.Mask)
       (net 2 +5V))
@@
       (net 1 GND))
     (pad 22 smd rect (at 4 -5.7 270) (size 1.5 0.55) (layers B.Cu B.Paste B.Mask)
-      (net 36 "Net-(U1-Pad22)"))
+      (net 32 "Net-(U1-Pad22)"))
     (pad 21 smd rect (at 3.2 -5.7 270) (size 1.5 0.55) (layers B.Cu B.Paste B.Mask)
-      (net 37 "Net-(U1-Pad21)"))
+      (net 33 "Net-(U1-Pad21)"))
     (pad 20 smd rect (at 2.4 -5.7 270) (size 1.5 0.55) (layers B.Cu B.Paste B.Mask)
-      (net 38 "Net-(U1-Pad20)"))
+      (net 34 "Net-(U1-Pad20)"))
     (pad 19 smd rect (at 1.6 -5.7 270) (size 1.5 0.55) (layers B.Cu B.Paste B.Mask)
-      (net 39 "Net-(U1-Pad19)"))
+      (net 35 "Net-(U1-Pad19)"))
     (pad 18 smd rect (at 0.8 -5.7 270) (size 1.5 0.55) (layers B.Cu B.Paste B.Mask)
-      (net 40 "Net-(U1-Pad18)"))
+      (net 36 "Net-(U1-Pad18)"))
     (pad 17 smd rect (at 0 -5.7 270) (size 1.5 0.55) (layers B.Cu B.Paste B.Mask)
       (net 3 "Net-(C4-Pad1)"))
@@
       (net 19 "Net-(R3-Pad2)"))
     (pad 12 smd rect (at -4 -5.7 270) (size 1.5 0.55) (layers B.Cu B.Paste B.Mask)
-      (net 41 "Net-(U1-Pad12)"))
+      (net 37 "Net-(U1-Pad12)"))
     (pad 11 smd rect (at -5.7 -4) (size 1.5 0.55) (layers B.Cu B.Paste B.Mask)
-      (net 42 "Net-(U1-Pad11)"))
+      (net 38 "Net-(U1-Pad11)"))
     (pad 10 smd rect (at -5.7 -3.2) (size 1.5 0.55) (layers B.Cu B.Paste B.Mask)
-      (net 43 "Net-(U1-Pad10)"))
+      (net 39 "Net-(U1-Pad10)"))
     (pad 9 smd rect (at -5.7 -2.4) (size 1.5 0.55) (layers B.Cu B.Paste B.Mask)
-      (net 44 "Net-(U1-Pad9)"))
+      (net 40 "Net-(U1-Pad9)"))
     (pad 8 smd rect (at -5.7 -1.6) (size 1.5 0.55) (layers B.Cu B.Paste B.Mask)
-      (net 45 "Net-(U1-Pad8)"))
+      (net 41 "Net-(U1-Pad8)"))
     (pad 7 smd rect (at -5.7 -0.8) (size 1.5 0.55) (layers B.Cu B.Paste B.Mask)
       (net 2 +5V))
@@
       (net 2 +5V))
     (pad 1 smd rect (at -5.7 4) (size 1.5 0.55) (layers B.Cu B.Paste B.Mask)
-      (net 46 "Net-(U1-Pad1)"))
+      (net 42 "Net-(U1-Pad1)"))
     (model ${KISYS3DMOD}/Package_QFP.3dshapes/TQFP-44_10x10mm_P0.8mm.wrl
       (at (xyz 0 0 0))
@@
   (segment (start 97.764501 91.477001) (end 97.764501 108.672999) (width 0.254) (layer B.Cu) (net 7))
   (segment (start 96.8375 90.55) (end 97.764501 91.477001) (width 0.254) (layer B.Cu) (net 7))
+  (segment (start 96.166599 110.270901) (end 96.8375 109.6) (width 0.254) (layer B.Cu) (net 7))
+  (segment (start 84.361939 110.270901) (end 96.166599 110.270901) (width 0.254) (layer B.Cu) (net 7))
+  (segment (start 78.046788 103.95575) (end 84.361939 110.270901) (width 0.254) (layer B.Cu) (net 7))
+  (segment (start 72.91475 103.95575) (end 78.046788 103.95575) (width 0.254) (layer B.Cu) (net 7))
   (segment (start 113.3 87.25) (end 110.45 84.4) (width 0.254) (layer B.Cu) (net 8))
   (segment (start 115.8875 87.25) (end 113.3 87.25) (width 0.254) (layer B.Cu) (net 8))
@@
   (segment (start 115.8875 108.896) (end 116.814501 107.968999) (width 0.254) (layer B.Cu) (net 9))
   (segment (start 115.8875 109.6) (end 115.8875 108.896) (width 0.254) (layer B.Cu) (net 9))
+  (segment (start 84.173882 110.724911) (end 114.762589 110.724911) (width 0.254) (layer B.Cu) (net 9))
+  (segment (start 78.204722 104.75575) (end 84.173882 110.724911) (width 0.254) (layer B.Cu) (net 9))
+  (segment (start 114.762589 110.724911) (end 115.8875 109.6) (width 0.254) (layer B.Cu) (net 9))
+  (segment (start 72.91475 104.75575) (end 78.204722 104.75575) (width 0.254) (layer B.Cu) (net 9))
   (segment (start 94.25 106.3) (end 91.4 103.45) (width 0.254) (layer B.Cu) (net 10))
   (segment (start 96.8375 106.3) (end 94.25 106.3) (width 0.254) (layer B.Cu) (net 10))
@@
   (segment (start 115.8875 106.3) (end 113.8625 106.3) (width 0.254) (layer B.Cu) (net 11))
   (segment (start 85.09 86.36) (end 104.14 86.36) (width 0.254) (layer F.Cu) (net 13))
+  (segment (start 76.281768 102.35575) (end 85.09 93.547518) (width 0.254) (layer B.Cu) (net 13))
+  (segment (start 85.09 93.547518) (end 85.09 86.36) (width 0.254) (layer B.Cu) (net 13))
+  (segment (start 72.91475 102.35575) (end 76.281768 102.35575) (width 0.254) (layer B.Cu) (net 13))
   (segment (start 104.0825 105.41) (end 104.14 105.4675) (width 0.254) (layer F.Cu) (net 14))
   (segment (start 85.09 105.41) (end 104.0825 105.41) (width 0.254) (layer F.Cu) (net 14))
+  (segment (start 82.83575 103.15575) (end 85.09 105.41) (width 0.254) (layer B.Cu) (net 14))
+  (segment (start 72.91475 103.15575) (end 82.83575 103.15575) (width 0.254) (layer B.Cu) (net 14))
   (segment (start 60.749352 93.37675) (end 64.01475 96.642148) (width 0.254) (layer B.Cu) (net 19))
   (segment (start 58.87975 93.37675) (end 60.749352 93.37675) (width 0.254) (layer B.Cu) (net 19))
